Commit message: Major changes to project based on real world condition

File: description/gazebo_controls.xacro (robot description, xacro)
@@ -2,5 +2,6 @@
 <robot xmlns:xacro="http://www.ros.org/wiki/xacro">
     <gazebo>
-        <plugin filename="libignition-gazebo-diff-drive-system.so" name="ignition::gazebo::systems::DiffDrive">
+        <!-- Harmonic naming: gz-sim-*-system / gz::sim::systems::* -->
+        <plugin filename="gz-sim-diff-drive-system" name="gz::sim::systems::DiffDrive">
             <!-- Wheel joints: two per side for the 4-wheel skid-steer -->
             <left_joint>l_f_wheel_joint</left_joint>
@@ -19,5 +20,6 @@
             <max_angular_velocity>1</max_angular_velocity>
             <min_angular_velocity>-1</min_angular_velocity>
-            <!-- Output -->
+            <!-- Output (wheel odometry; whether it is fused or discarded is
+                 still an open decision, pending the sensor-set question) -->
             <odom_publish_frequency>50</odom_publish_frequency>
             <topic>cmd_vel</topic>
@@ -27,5 +29,5 @@
             <child_frame_id>base_link</child_frame_id>
         </plugin>
-        <plugin filename="libignition-gazebo-joint-state-publisher-system.so" name="ignition::gazebo::systems::JointStatePublisher">
+        <plugin filename="gz-sim-joint-state-publisher-system" name="gz::sim::systems::JointStatePublisher">
             <topic>joint_states</topic>
         </plugin>

File: description/gazebo_materials.xacro (robot description, xacro)
@@ -10,6 +10,6 @@
          kept high for straight-line traction; mu2 (lateral, local Y) lowered
          so wheels can slide sideways during a skid-steer pivot without
-         stick-slip. kp/kd soften contact stiffness slightly to reduce
-         numerical jitter. Starting values — tune mu2 down further (e.g. 0.15)
+         stick-slip. kp/kd are ODE-only (ignored by DART, the Harmonic
+         default engine) and kept only in case you switch engines. Starting values — tune mu2 down further (e.g. 0.15)
          if rocking persists, or up if the robot starts sliding out during
          normal turns. -->
@@ -70,5 +70,5 @@
         </material>
     </gazebo>
-    <gazebo reference="f_rgbd_link">
+    <gazebo reference="f_camera_link">
         <material>
             <ambient>0 1 0 1</ambient>
@@ -76,5 +76,5 @@
         </material>
     </gazebo>
-    <gazebo reference="r_rgbd_link">
+    <gazebo reference="r_camera_link">
         <material>
             <ambient>0 1 0 1</ambient>
@@ -82,14 +82,8 @@
         </material>
     </gazebo>
-    <gazebo reference="f_lidar_link">
+    <gazebo reference="gps_link">
         <material>
-            <ambient>0 0 1 1</ambient>
-            <diffuse>0 0 1 1</diffuse>
-        </material>
-    </gazebo>
-    <gazebo reference="r_lidar_link">
-        <material>
-            <ambient>0 0 1 1</ambient>
-            <diffuse>0 0 1 1</diffuse>
+            <ambient>1 0 0 1</ambient>
+            <diffuse>1 0 0 1</diffuse>
         </material>
     </gazebo>

File: description/gazebo_sensors.xacro (robot description, xacro)
@@ -1,132 +1,91 @@
 <?xml version="1.0"?>
 <robot xmlns:xacro="http://www.ros.org/wiki/xacro">
+    <!-- Sensor set: 2x monocular camera (130 deg HFOV), 1x IMU, 1x GPS. Nothing else.
+         Requires in the world: Sensors (ogre2), Imu, NavSat systems, and
+         <spherical_coordinates> (see worlds/outdoor_flat.world). -->
+    <xacro:property name="cam_hfov" value="2.2689"/>   <!-- 130 deg in rad -->
+    <xacro:property name="cam_w" value="640"/>
+    <xacro:property name="cam_h" value="480"/>
+    <xacro:property name="cam_rate" value="20"/>
+    <!-- Plain rectilinear (pinhole) projection: no lens distortion is modeled,
+         so a 130 deg image is heavily stretched at the edges. Switch to a
+         distortion/fisheye model once the VSLAM framework is chosen. -->
+    <xacro:macro name="mono_camera" params="side link optical_link">
+        <gazebo reference="${link}">
+            <sensor name="${side}_camera" type="camera">
+                <pose>0.05 0 0 0 0 0</pose>
+                <always_on>true</always_on>
+                <visualize>false</visualize>
+                <update_rate>${cam_rate}</update_rate>
+                <topic>camera/${side}/image</topic>
+                <gz_frame_id>${optical_link}</gz_frame_id>
+                <camera name="${side}_camera">
+                    <horizontal_fov>${cam_hfov}</horizontal_fov>
+                    <image>
+                        <width>${cam_w}</width>
+                        <height>${cam_h}</height>
+                        <format>R8G8B8</format>
+                    </image>
+                    <clip>
+                        <near>0.1</near>
+                        <far>100.0</far>
+                    </clip>
+                    <noise>
+                        <type>gaussian</type>
+                        <mean>0.0</mean>
+                        <stddev>0.007</stddev>
+                    </noise>
+                    <camera_info_topic>camera/${side}/camera_info</camera_info_topic>
+                </camera>
+            </sensor>
+        </gazebo>
+    </xacro:macro>
+    <xacro:mono_camera side="front" link="f_camera_link" optical_link="f_camera_optical_link"/>
+    <xacro:mono_camera side="rear"  link="r_camera_link" optical_link="r_camera_optical_link"/>
     <!-- =========================================== -->
-    <!-- ========== FRONT CAMERA SENSORS ============ -->
+    <!-- ==================== IMU ================== -->
     <!-- =========================================== -->
-    <gazebo reference="f_rgbd_link">
-        <sensor name="rgbd_camera" type="rgbd_camera">
-            <pose>0.05 0 0 0 0 0</pose>
+    <!-- Noise values are typical MEMS-grade starting points; replace with the
+         datasheet of the real IMU for the Jetson/VIO tuning. -->
+    <gazebo reference="imu_link">
+        <sensor name="imu" type="imu">
             <always_on>true</always_on>
-            <visualize>true</visualize>
-            <update_rate>20</update_rate>
-            <topic>camera/front</topic>
-            <gz_frame_id>f_rgbd_link</gz_frame_id>
-            <camera name="rgbd_camera">
-                <horizontal_fov>1.089</horizontal_fov>
-                <image>
-                    <width>640</width>
-                    <height>480</height>
-                    <format>R8G8B8</format>
-                </image>
-                <clip>
-                    <near>0.05</near>
-                    <far>20.0</far>
-                </clip>
-                <camera_info_topic>camera/front/camera_info</camera_info_topic>
-                <depth_camera>
-                    <clip>
-                        <near>0.05</near>
-                        <far>10.0</far>
-                    </clip>
-                </depth_camera>
-            </camera>
+            <visualize>false</visualize>
+            <update_rate>200</update_rate>
+            <topic>imu</topic>
+            <gz_frame_id>imu_link</gz_frame_id>
+            <imu>
+                <angular_velocity>
+                    <x><noise type="gaussian"><mean>0</mean><stddev>2e-4</stddev><bias_mean>7.5e-6</bias_mean><bias_stddev>8e-7</bias_stddev></noise></x>
+                    <y><noise type="gaussian"><mean>0</mean><stddev>2e-4</stddev><bias_mean>7.5e-6</bias_mean><bias_stddev>8e-7</bias_stddev></noise></y>
+                    <z><noise type="gaussian"><mean>0</mean><stddev>2e-4</stddev><bias_mean>7.5e-6</bias_mean><bias_stddev>8e-7</bias_stddev></noise></z>
+                </angular_velocity>
+                <linear_acceleration>
+                    <x><noise type="gaussian"><mean>0</mean><stddev>1.7e-2</stddev><bias_mean>0.1</bias_mean><bias_stddev>1e-3</bias_stddev></noise></x>
+                    <y><noise type="gaussian"><mean>0</mean><stddev>1.7e-2</stddev><bias_mean>0.1</bias_mean><bias_stddev>1e-3</bias_stddev></noise></y>
+                    <z><noise type="gaussian"><mean>0</mean><stddev>1.7e-2</stddev><bias_mean>0.1</bias_mean><bias_stddev>1e-3</bias_stddev></noise></z>
+                </linear_acceleration>
+            </imu>
         </sensor>
     </gazebo>
     <!-- =========================================== -->
-    <!-- =========== REAR CAMERA SENSOR ============ -->
+    <!-- ==================== GPS ================== -->
     <!-- =========================================== -->
-    <gazebo reference="r_rgbd_link">
-        <sensor name="camera2_rgbd" type="rgbd_camera">
-            <pose>0.05 0 0 0 0 0</pose>
+    <gazebo reference="gps_link">
+        <sensor name="navsat" type="navsat">
             <always_on>true</always_on>
-            <visualize>true</visualize>
-            <update_rate>20</update_rate>
-            <topic>camera/rear</topic>
-            <gz_frame_id>r_rgbd_link</gz_frame_id>
-            <camera name="rgbd_camera">
-                <horizontal_fov>1.089</horizontal_fov>
-                <image>
-                    <width>640</width>
-                    <height>480</height>
-                    <format>R8G8B8</format>
-                </image>
-                <clip>
-                    <near>0.05</near>
-                    <far>20.0</far>
-                </clip>
-                <camera_info_topic>camera/rear/camera_info</camera_info_topic>
-                <depth_camera>
-                    <clip>
-                        <near>0.05</near>
-                        <far>10.0</far>
-                    </clip>
-                </depth_camera>
-            </camera>
-        </sensor>
-    </gazebo>
-    <!-- =========================================== -->
-    <!-- ========== FRONT LIDAR SENSOR ============= -->
-    <!-- =========================================== -->
-    <gazebo reference="f_lidar_link">
-        <sensor name="front_lidar" type="gpu_lidar">
-            <pose>0 0 0 0 0 0</pose>
-            <visualize>true</visualize>
             <update_rate>10</update_rate>
-            <topic>lidar/front/scan</topic>
-            <gz_frame_id>f_lidar_link</gz_frame_id>
-            <lidar>
-                <scan>
+            <topic>gps/fix</topic>
+            <gz_frame_id>gps_link</gz_frame_id>
+            <navsat>
+                <position_sensing>
                     <horizontal>
-                        <samples>240</samples>
-                        <resolution>1</resolution>
-                        <min_angle>-2.193</min_angle>
-                        <max_angle>2.193</max_angle>
+                        <noise type="gaussian"><mean>0</mean><stddev>1.0</stddev></noise>
                     </horizontal>
                     <vertical>
-                        <samples>16</samples>
-                        <resolution>1</resolution>
-                        <min_angle>-0.1</min_angle>
-                        <max_angle>0.179</max_angle>
+                        <noise type="gaussian"><mean>0</mean><stddev>2.0</stddev></noise>
                     </vertical>
-                </scan>
-                <range>
-                    <min>0.3</min>
-                    <max>12.0</max>
-                    <resolution>0.01</resolution>
-                </range>
-            </lidar>
-        </sensor>
-    </gazebo>
-    <!-- =========================================== -->
-    <!-- ========== REAR LIDAR SENSOR =============== -->
-    <!-- =========================================== -->
-    <gazebo reference="r_lidar_link">
-        <sensor name="rear_lidar" type="gpu_lidar">
-            <pose>0 0 0 0 0 0</pose>
-            <visualize>true</visualize>
-            <update_rate>10</update_rate>
-            <topic>lidar/rear/scan</topic>
-            <gz_frame_id>r_lidar_link</gz_frame_id>
-            <lidar>
-                <scan>
-                    <horizontal>
-                        <samples>240</samples>
-                        <resolution>1</resolution>
-                        <min_angle>-2.193</min_angle>
-                        <max_angle>2.193</max_angle>
-                    </horizontal>
-                    <vertical>
-                        <samples>16</samples>
-                        <resolution>1</resolution>
-                        <min_angle>-0.1</min_angle>
-                        <max_angle>0.179</max_angle>
-                    </vertical>
-                </scan>
-                <range>
-                    <min>0.3</min>
-                    <max>12.0</max>
-                    <resolution>0.01</resolution>
-                </range>
-            </lidar>
+                </position_sensing>
+            </navsat>
         </sensor>
     </gazebo>

File: description/joints.xacro (robot description, xacro)
@@ -49,28 +49,43 @@
     </joint>
     <!-- =========================================== -->
-    <!-- ================ CAMERA JOINTS ============ -->
+    <!-- ================ MONO CAMERA JOINTS ============ -->
     <!-- =========================================== -->
-    <joint name="f_rgbd_joint" type="fixed">
+    <joint name="f_camera_joint" type="fixed">
         <origin xyz="0.6525 0.0 0.6625" rpy="0 0 0"/>
         <parent link="base_link"/>
-        <child link="f_rgbd_link"/>
+        <child link="f_camera_link"/>
     </joint>
-    <joint name="r_rgbd_joint" type="fixed">
+    <joint name="r_camera_joint" type="fixed">
         <origin xyz="-0.6525 0.0 0.6625" rpy="0 0 ${pi}"/>
         <parent link="base_link"/>
-        <child link="r_rgbd_link"/>
+        <child link="r_camera_link"/>
+    </joint>
+    <!-- Optical frames: sit at the lens (matches the 0.05 m sensor <pose> in
+         gazebo_sensors.xacro) with REP-103 axis rotation. -->
+    <joint name="f_camera_optical_joint" type="fixed">
+        <origin xyz="0.05 0 0" rpy="${-pi/2} 0 ${-pi/2}"/>
+        <parent link="f_camera_link"/>
+        <child link="f_camera_optical_link"/>
+    </joint>
+    <joint name="r_camera_optical_joint" type="fixed">
+        <origin xyz="0.05 0 0" rpy="${-pi/2} 0 ${-pi/2}"/>
+        <parent link="r_camera_link"/>
+        <child link="r_camera_optical_link"/>
     </joint>
     <!-- =========================================== -->
-    <!-- ================ LIDAR JOINTS ============= -->
+    <!-- ============== IMU + GPS JOINTS =========== -->
     <!-- =========================================== -->
-    <joint name="f_lidar_joint" type="fixed">
-        <origin xyz="0.55 0.0 0.74" rpy="0 0 0"/>
+    <!-- IMU near the whole-robot CoM (base_link inertial origin). -->
+    <joint name="imu_joint" type="fixed">
+        <origin xyz="0 0 0.486" rpy="0 0 0"/>
         <parent link="base_link"/>
-        <child link="f_lidar_link"/>
+        <child link="imu_link"/>
     </joint>
-    <joint name="r_lidar_joint" type="fixed">
-        <origin xyz="-0.55 0.0 0.74" rpy="0 0 ${pi}"/>
+    <!-- GPS antenna on top of the chassis (top face is z = 0.636), slightly
+         aft so it clears the cameras' view. -->
+    <joint name="gps_joint" type="fixed">
+        <origin xyz="-0.2 0 0.636" rpy="0 0 0"/>
         <parent link="base_link"/>
-        <child link="r_lidar_link"/>
+        <child link="gps_link"/>
     </joint>
 </robot>

File: description/links.xacro (robot description, xacro)
@@ -17,18 +17,4 @@
             <material name="desert_tan"/>
         </visual>
-        <visual>
-    	    <origin xyz="0.55 0.0 0.685" rpy="0 0 0"/>
-            <geometry>
-                <cylinder radius="0.05" length="0.1"/>
-            </geometry>
-            <material name="desert_tan"/>
-        </visual>
-         <visual>
-    	    <origin xyz="-0.55 0.0 0.685" rpy="0 0 0"/>
-            <geometry>
-                <cylinder radius="0.05" length="0.1"/>
-            </geometry>
-            <material name="desert_tan"/>
-        </visual>
         <collision>
             <origin xyz="0.000973 0.000007 0.486096" rpy="0 0 0"/>
@@ -177,7 +163,7 @@
     </link>
     <!-- =========================================== -->
-    <!-- ========== FRONT RGBD CAMERA ============== -->
-    <!-- =========================================== -->
-    <link name="f_rgbd_link">
+    <!-- ========== FRONT MONO CAMERA ============== -->
+    <!-- =========================================== -->
+    <link name="f_camera_link">
         <inertial>
             <origin xyz="0 0 0.0225" rpy="0 0 0"/>
@@ -211,7 +197,7 @@
     </link>
     <!-- =========================================== -->
-    <!-- =========== REAR RGBD CAMERA ============== -->
-    <!-- =========================================== -->
-    <link name="r_rgbd_link">
+    <!-- =========== REAR MONO CAMERA ============== -->
+    <!-- =========================================== -->
+    <link name="r_camera_link">
         <inertial>
             <origin xyz="0 0 0.0225" rpy="0 0 0"/>
@@ -244,49 +230,34 @@
         </collision>
   </link>
-    <!-- =========================================== -->
-    <!-- ========== FRONT LIVOX LIDAR ============== -->
-    <!-- =========================================== -->
-    <link name="f_lidar_link">
-        <inertial>
-            <origin xyz="0 0 0.0375" rpy="0 0 0"/>
-            <mass value="1.0750137361502572"/>
-            <inertia ixx="0.001176" iyy="0.001176" izz="0.001344" ixy="0.0" iyz="0.0" ixz="0.0"/>
-        </inertial>
-        <visual>
-            <origin xyz="0 0 0.0375" rpy="0 0 0"/>
-            <geometry>
-                <cylinder radius="0.05" length="0.075"/>
-            </geometry>
-            <material name="blue"/>
-        </visual>
-        <collision>
-            <origin xyz="0 0 0.0375" rpy="0 0 0"/>
-            <geometry>
-                <cylinder radius="0.05" length="0.075"/>
-            </geometry>
-        </collision>
-    </link>
-    <!-- =========================================== -->
-    <!-- =========== REAR LIVOX LIDAR =============== -->
-    <!-- =========================================== -->
-    <link name="r_lidar_link">
-        <inertial>
-            <origin xyz="0 0 0.0375" rpy="0 0 0"/>
-            <mass value="1.0750137361502572"/>
-            <inertia ixx="0.001176" iyy="0.001176" izz="0.001344" ixy="0.0" iyz="0.0" ixz="0.0"/>
-        </inertial>
-        <visual>
-            <origin xyz="0 0 0.0375" rpy="0 0 0"/>
-            <geometry>
-                <cylinder radius="0.05" length="0.075"/>
-            </geometry>
-            <material name="blue"/>
-        </visual>
-        <collision>
-            <origin xyz="0 0 0.0375" rpy="0 0 0"/>
-            <geometry>
-                <cylinder radius="0.05" length="0.075"/>
-            </geometry>
-        </collision>
+    <!-- Optical frames (REP-103: z forward, x right, y down). Empty frames;
+         images/camera_info are stamped with these so VSLAM gets the right axes. -->
+    <link name="f_camera_optical_link"/>
+    <link name="r_camera_optical_link"/>
+    <!-- =========================================== -->
+    <!-- ================== IMU ==================== -->
+    <!-- =========================================== -->
+    <link name="imu_link">
+        <inertial>
+            <origin xyz="0 0 0" rpy="0 0 0"/>
+            <mass value="0.05"/>
+            <inertia ixx="1e-5" iyy="1e-5" izz="1e-5" ixy="0.0" iyz="0.0" ixz="0.0"/>
+        </inertial>
+    </link>
+    <!-- =========================================== -->
+    <!-- ================== GPS ==================== -->
+    <!-- =========================================== -->
+    <link name="gps_link">
+        <inertial>
+            <origin xyz="0 0 0.01" rpy="0 0 0"/>
+            <mass value="0.1"/>
+            <inertia ixx="2e-5" iyy="2e-5" izz="2e-5" ixy="0.0" iyz="0.0" ixz="0.0"/>
+        </inertial>
+        <visual>
+            <origin xyz="0 0 0.01" rpy="0 0 0"/>
+            <geometry>
+                <cylinder radius="0.04" length="0.02"/>
+            </geometry>
+            <material name="red"/>
+        </visual>
     </link>
 </robot>
