Commit message: major change to project #3

File: description/gazebo_controls.xacro (robot description, xacro)
@@ -2,24 +2,21 @@
 <robot xmlns:xacro="http://www.ros.org/wiki/xacro">
     <gazebo>
-        <!-- Harmonic naming: gz-sim-*-system / gz::sim::systems::* -->
-        <plugin filename="gz-sim-diff-drive-system" name="gz::sim::systems::DiffDrive">
-            <!-- Wheel joints: two per side for the 4-wheel skid-steer -->
-            <left_joint>l_f_wheel_joint</left_joint>
-            <left_joint>l_r_wheel_joint</left_joint>
-            <right_joint>r_f_wheel_joint</right_joint>
-            <right_joint>r_r_wheel_joint</right_joint>
-            <!-- Wheel geometry -->
-            <wheel_separation>0.874</wheel_separation>
-            <wheel_radius>0.225</wheel_radius>
-            <max_linear_acceleration>0.5</max_linear_acceleration>
-            <min_linear_acceleration>-0.5</min_linear_acceleration>
-            <max_angular_acceleration>1</max_angular_acceleration>
-            <min_angular_acceleration>-1</min_angular_acceleration>
-            <max_linear_velocity>2</max_linear_velocity>
-            <min_linear_velocity>-2</min_linear_velocity>
-            <max_angular_velocity>1</max_angular_velocity>
-            <min_angular_velocity>-1</min_angular_velocity>
-            <!-- Output (wheel odometry; whether it is fused or discarded is
-                 still an open decision, pending the sensor-set question) -->
+        <plugin filename="libignition-gazebo-diff-drive-system.so" name="ignition::gazebo::systems::DiffDrive">
+            <!-- True 2-wheel differential drive (front caster is passive) -->
+            <left_joint>l_wheel_joint</left_joint>
+            <right_joint>r_wheel_joint</right_joint>
+            <!-- Wheel geometry (shared with properties.xacro) -->
+            <wheel_separation>${wheel_separation}</wheel_separation>
+            <wheel_radius>${wheel_radius}</wheel_radius>
+            <!-- Limits scaled for a small indoor robot -->
+            <max_linear_acceleration>1.0</max_linear_acceleration>
+            <min_linear_acceleration>-1.0</min_linear_acceleration>
+            <max_angular_acceleration>2.0</max_angular_acceleration>
+            <min_angular_acceleration>-2.0</min_angular_acceleration>
+            <max_linear_velocity>1.0</max_linear_velocity>
+            <min_linear_velocity>-1.0</min_linear_velocity>
+            <max_angular_velocity>2.0</max_angular_velocity>
+            <min_angular_velocity>-2.0</min_angular_velocity>
+            <!-- Output -->
             <odom_publish_frequency>50</odom_publish_frequency>
             <topic>cmd_vel</topic>
@@ -29,5 +26,5 @@
             <child_frame_id>base_link</child_frame_id>
         </plugin>
-        <plugin filename="gz-sim-joint-state-publisher-system" name="gz::sim::systems::JointStatePublisher">
+        <plugin filename="libignition-gazebo-joint-state-publisher-system.so" name="ignition::gazebo::systems::JointStatePublisher">
             <topic>joint_states</topic>
         </plugin>

File: description/gazebo_materials.xacro (robot description, xacro)
@@ -7,68 +7,38 @@
         </material>
     </gazebo>
-    <!-- Anisotropic wheel friction: mu1 (fdir1 = rolling direction, local X)
-         kept high for straight-line traction; mu2 (lateral, local Y) lowered
-         so wheels can slide sideways during a skid-steer pivot without
-         stick-slip. kp/kd are ODE-only (ignored by DART, the Harmonic
-         default engine) and kept only in case you switch engines. Starting values — tune mu2 down further (e.g. 0.15)
-         if rocking persists, or up if the robot starts sliding out during
-         normal turns. -->
-    <gazebo reference="l_f_wheel_link">
+    <!-- Drive wheels: with only two driven wheels + a caster there is no
+         skid-steer scrubbing, so lateral friction should be HIGH (mu2 = mu1).
+         The anisotropic low-mu2 setting from the 4-wheel bot would let the
+         small robot slide sideways. kp/kd soften contact slightly. -->
+    <xacro:macro name="wheel_surface" params="prefix">
+        <gazebo reference="${prefix}_wheel_link">
+            <material>
+                <ambient>0 0 0 1</ambient>
+                <diffuse>0 0 0 1</diffuse>
+            </material>
+            <mu1>1.0</mu1>
+            <mu2>1.0</mu2>
+            <kp>1e6</kp>
+            <kd>1.0</kd>
+        </gazebo>
+    </xacro:macro>
+    <xacro:wheel_surface prefix="l"/>
+    <xacro:wheel_surface prefix="r"/>
+    <!-- Caster: near-frictionless so it never drags or biases turns. -->
+    <gazebo reference="caster_link">
         <material>
-            <ambient>0 0 0 1</ambient>
-            <diffuse>0 0 0 1</diffuse>
+            <ambient>0.5 0.5 0.5 1</ambient>
+            <diffuse>0.5 0.5 0.5 1</diffuse>
         </material>
-        <mu1>1.0</mu1>
-        <mu2>0.3</mu2>
-        <fdir1>1 0 0</fdir1>
-        <kp>1e6</kp>
-        <kd>10</kd>
+        <mu1>0.01</mu1>
+        <mu2>0.01</mu2>
     </gazebo>
-    <gazebo reference="l_r_wheel_link">
+    <gazebo reference="stereo_bar_link">
         <material>
-            <ambient>0 0 0 1</ambient>
-            <diffuse>0 0 0 1</diffuse>
-        </material>
-        <mu1>1.0</mu1>
-        <mu2>0.3</mu2>
-        <fdir1>1 0 0</fdir1>
-        <kp>1e6</kp>
-        <kd>10</kd>
-    </gazebo>
-    <gazebo reference="r_f_wheel_link">
-        <material>
-            <ambient>0 0 0 1</ambient>
-            <diffuse>0 0 0 1</diffuse>
-        </material>
-        <mu1>1.0</mu1>
-        <mu2>0.3</mu2>
-        <fdir1>1 0 0</fdir1>
-        <kp>1e6</kp>
-        <kd>10</kd>
-    </gazebo>
-    <gazebo reference="r_r_wheel_link">
-        <material>
-            <ambient>0 0 0 1</ambient>
-            <diffuse>0 0 0 1</diffuse>
-        </material>
-        <mu1>1.0</mu1>
-        <mu2>0.3</mu2>
-        <fdir1>1 0 0</fdir1>
-        <kp>1e6</kp>
-        <kd>10</kd>
-    </gazebo>
-    <gazebo reference="front_bumper_link">
-        <material>
-            <ambient>1 1 1 1</ambient>
-            <diffuse>1 1 1 1</diffuse>
+            <ambient>0.5 0.5 0.5 1</ambient>
+            <diffuse>0.5 0.5 0.5 1</diffuse>
         </material>
     </gazebo>
-    <gazebo reference="rear_bumper_link">
-        <material>
-            <ambient>1 1 1 1</ambient>
-            <diffuse>1 1 1 1</diffuse>
-        </material>
-    </gazebo>
-    <gazebo reference="f_camera_link">
+    <gazebo reference="cam_left_link">
         <material>
             <ambient>0 1 0 1</ambient>
@@ -76,5 +46,5 @@
         </material>
     </gazebo>
-    <gazebo reference="r_camera_link">
+    <gazebo reference="cam_right_link">
         <material>
             <ambient>0 1 0 1</ambient>
@@ -82,5 +52,5 @@
         </material>
     </gazebo>
-    <gazebo reference="gps_link">
+    <gazebo reference="imu_link">
         <material>
             <ambient>1 0 0 1</ambient>
@@ -88,3 +58,9 @@
         </material>
     </gazebo>
+    <gazebo reference="gps_link">
+        <material>
+            <ambient>0 0 1 1</ambient>
+            <diffuse>0 0 1 1</diffuse>
+        </material>
+    </gazebo>
 </robot>

File: description/gazebo_sensors.xacro (robot description, xacro)
@@ -1,38 +1,34 @@
 <?xml version="1.0"?>
 <robot xmlns:xacro="http://www.ros.org/wiki/xacro">
-    <!-- Sensor set: 2x monocular camera (130 deg HFOV), 1x IMU, 1x GPS. Nothing else.
-         Requires in the world: Sensors (ogre2), Imu, NavSat systems, and
-         <spherical_coordinates> (see worlds/outdoor_flat.world). -->
-    <xacro:property name="cam_hfov" value="2.2689"/>   <!-- 130 deg in rad -->
-    <xacro:property name="cam_w" value="640"/>
-    <xacro:property name="cam_h" value="480"/>
-    <xacro:property name="cam_rate" value="20"/>
-    <!-- Plain rectilinear (pinhole) projection: no lens distortion is modeled,
-         so a 130 deg image is heavily stretched at the edges. Switch to a
-         distortion/fisheye model once the VSLAM framework is chosen. -->
-    <xacro:macro name="mono_camera" params="side link optical_link">
-        <gazebo reference="${link}">
-            <sensor name="${side}_camera" type="camera">
-                <pose>0.05 0 0 0 0 0</pose>
+    <!-- =========================================== -->
+    <!-- ============ STEREO CAMERA PAIR =========== -->
+    <!-- =========================================== -->
+    <!-- Plain `camera` sensors (not the combined rgbd_camera), which avoids
+         the ogre2 corruption bug from ros_gz#738. Image/camera_info headers
+         use the optical frame. Left camera is always on; the right one is
+         dropped when launched with stereo_mode:=mono. -->
+    <xacro:macro name="camera_sensor" params="side">
+        <gazebo reference="cam_${side}_link">
+            <sensor name="cam_${side}" type="camera">
                 <always_on>true</always_on>
-                <visualize>false</visualize>
-                <update_rate>${cam_rate}</update_rate>
+                <visualize>${sensor_visualize}</visualize>
+                <update_rate>${camera_rate}</update_rate>
                 <topic>camera/${side}/image</topic>
-                <gz_frame_id>${optical_link}</gz_frame_id>
-                <camera name="${side}_camera">
-                    <horizontal_fov>${cam_hfov}</horizontal_fov>
+                <gz_frame_id>cam_${side}_optical_frame</gz_frame_id>
+                <camera name="cam_${side}">
+                    <horizontal_fov>${camera_hfov}</horizontal_fov>
                     <image>
-                        <width>${cam_w}</width>
-                        <height>${cam_h}</height>
+                        <width>${camera_width}</width>
+                        <height>${camera_height}</height>
                         <format>R8G8B8</format>
                     </image>
                     <clip>
-                        <near>0.1</near>
-                        <far>100.0</far>
+                        <near>0.05</near>
+                        <far>30.0</far>
                     </clip>
                     <noise>
                         <type>gaussian</type>
                         <mean>0.0</mean>
-                        <stddev>0.007</stddev>
+                        <stddev>${camera_noise_stddev}</stddev>
                     </noise>
                     <camera_info_topic>camera/${side}/camera_info</camera_info_topic>
@@ -41,28 +37,29 @@
         </gazebo>
     </xacro:macro>
-    <xacro:mono_camera side="front" link="f_camera_link" optical_link="f_camera_optical_link"/>
-    <xacro:mono_camera side="rear"  link="r_camera_link" optical_link="r_camera_optical_link"/>
+    <xacro:camera_sensor side="left"/>
+    <xacro:if value="$(arg enable_right_camera)">
+        <xacro:camera_sensor side="right"/>
+    </xacro:if>
     <!-- =========================================== -->
     <!-- ==================== IMU ================== -->
     <!-- =========================================== -->
-    <!-- Noise values are typical MEMS-grade starting points; replace with the
-         datasheet of the real IMU for the Jetson/VIO tuning. -->
+    <!-- Needs the Imu system plugin in the world file. -->
     <gazebo reference="imu_link">
         <sensor name="imu" type="imu">
             <always_on>true</always_on>
             <visualize>false</visualize>
-            <update_rate>200</update_rate>
+            <update_rate>${imu_rate}</update_rate>
             <topic>imu</topic>
             <gz_frame_id>imu_link</gz_frame_id>
             <imu>
                 <angular_velocity>
-                    <x><noise type="gaussian"><mean>0</mean><stddev>2e-4</stddev><bias_mean>7.5e-6</bias_mean><bias_stddev>8e-7</bias_stddev></noise></x>
-                    <y><noise type="gaussian"><mean>0</mean><stddev>2e-4</stddev><bias_mean>7.5e-6</bias_mean><bias_stddev>8e-7</bias_stddev></noise></y>
-                    <z><noise type="gaussian"><mean>0</mean><stddev>2e-4</stddev><bias_mean>7.5e-6</bias_mean><bias_stddev>8e-7</bias_stddev></noise></z>
+                    <x><noise type="gaussian"><mean>0.0</mean><stddev>2e-4</stddev></noise></x>
+                    <y><noise type="gaussian"><mean>0.0</mean><stddev>2e-4</stddev></noise></y>
+                    <z><noise type="gaussian"><mean>0.0</mean><stddev>2e-4</stddev></noise></z>
                 </angular_velocity>
                 <linear_acceleration>
-                    <x><noise type="gaussian"><mean>0</mean><stddev>1.7e-2</stddev><bias_mean>0.1</bias_mean><bias_stddev>1e-3</bias_stddev></noise></x>
-                    <y><noise type="gaussian"><mean>0</mean><stddev>1.7e-2</stddev><bias_mean>0.1</bias_mean><bias_stddev>1e-3</bias_stddev></noise></y>
-                    <z><noise type="gaussian"><mean>0</mean><stddev>1.7e-2</stddev><bias_mean>0.1</bias_mean><bias_stddev>1e-3</bias_stddev></noise></z>
+                    <x><noise type="gaussian"><mean>0.0</mean><stddev>1.7e-2</stddev></noise></x>
+                    <y><noise type="gaussian"><mean>0.0</mean><stddev>1.7e-2</stddev></noise></y>
+                    <z><noise type="gaussian"><mean>0.0</mean><stddev>1.7e-2</stddev></noise></z>
                 </linear_acceleration>
             </imu>
@@ -72,21 +69,16 @@
     <!-- ==================== GPS ================== -->
     <!-- =========================================== -->
-    <gazebo reference="gps_link">
-        <sensor name="navsat" type="navsat">
-            <always_on>true</always_on>
-            <update_rate>10</update_rate>
-            <topic>gps/fix</topic>
-            <gz_frame_id>gps_link</gz_frame_id>
-            <navsat>
-                <position_sensing>
-                    <horizontal>
-                        <noise type="gaussian"><mean>0</mean><stddev>1.0</stddev></noise>
-                    </horizontal>
-                    <vertical>
-                        <noise type="gaussian"><mean>0</mean><stddev>2.0</stddev></noise>
-                    </vertical>
-                </position_sensing>
-            </navsat>
-        </sensor>
-    </gazebo>
+    <!-- Toggle with enable_gps:=true. Meaningless in indoor worlds (no sky
+         view); intended for outdoor/yard-style maps. Needs the NavSat system
+         plugin and <spherical_coordinates> in the world file. -->
+    <xacro:if value="$(arg enable_gps)">
+        <gazebo reference="gps_link">
+            <sensor name="navsat" type="navsat">
+                <always_on>true</always_on>
+                <update_rate>${gps_rate}</update_rate>
+                <topic>navsat</topic>
+                <gz_frame_id>gps_link</gz_frame_id>
+            </sensor>
+        </gazebo>
+    </xacro:if>
 </robot>

File: description/joints.xacro (robot description, xacro)
@@ -2,88 +2,60 @@
 <robot xmlns:xacro="http://www.ros.org/wiki/xacro">
     <!-- =========================================== -->
-    <!-- ================ WHEEL JOINTS ============= -->
+    <!-- ============== DRIVE WHEELS =============== -->
     <!-- =========================================== -->
-    <joint name="l_f_wheel_joint" type="continuous">
-        <origin xyz="0.45 0.325 0.225" rpy="0 0 0"/>
+    <joint name="l_wheel_joint" type="continuous">
+        <origin xyz="0 ${wheel_y} 0" rpy="0 0 0"/>
         <parent link="base_link"/>
-        <child link="l_f_wheel_link"/>
-        <axis xyz="0.0 1.0 0.0"/>
-        <dynamics damping="1.0" friction="0.1"/>
+        <child link="l_wheel_link"/>
+        <axis xyz="0 1 0"/>
+        <dynamics damping="0.01" friction="0.01"/>
     </joint>
-    <joint name="l_r_wheel_joint" type="continuous">
-        <origin xyz="-0.45 0.325 0.225" rpy="0 0 0"/>
+    <joint name="r_wheel_joint" type="continuous">
+        <origin xyz="0 ${-wheel_y} 0" rpy="0 0 0"/>
         <parent link="base_link"/>
-        <child link="l_r_wheel_link"/>
-        <axis xyz="0.0 1.0 0.0"/>
-        <dynamics damping="1.0" friction="0.1"/>
-    </joint>
-    <joint name="r_r_wheel_joint" type="continuous">
-        <origin xyz="-0.45 -0.325 0.225" rpy="0 0 0"/>
-        <parent link="base_link"/>
-        <child link="r_r_wheel_link"/>
-        <axis xyz="0.0 1.0 0.0"/>
-        <dynamics damping="1.0" friction="0.1"/>
-    </joint>
-    <joint name="r_f_wheel_joint" type="continuous">
-        <origin xyz="0.45 -0.325 0.225" rpy="0 0 0"/>
-        <parent link="base_link"/>
-        <child link="r_f_wheel_link"/>
-        <axis xyz="0.0 1.0 0.0"/>
-        <dynamics damping="1.0" friction="0.1"/>
+        <child link="r_wheel_link"/>
+        <axis xyz="0 1 0"/>
+        <dynamics damping="0.01" friction="0.01"/>
     </joint>
     <!-- =========================================== -->
-    <!-- ================ BUMPER JOINTS ============ -->
+    <!-- ================= CASTER ================== -->
     <!-- =========================================== -->
-    <joint name="front_bumper_joint" type="fixed">
-        <origin xyz="0.7 0.225 0.45" rpy="0 0 0"/>
+    <joint name="caster_joint" type="fixed">
+        <origin xyz="${caster_x} 0 ${caster_z}" rpy="0 0 0"/>
         <parent link="base_link"/>
-        <child link="front_bumper_link"/>
-    </joint>
-    <!-- Mirrors front_bumper_joint across the YZ plane (X negated) to
-         counterbalance the front bumper's mass and pull the whole-robot
-         center of mass back toward base_link's origin. -->
-    <joint name="rear_bumper_joint" type="fixed">
-        <origin xyz="-0.7 0.225 0.45" rpy="0 0 0"/>
-        <parent link="base_link"/>
-        <child link="rear_bumper_link"/>
+        <child link="caster_link"/>
     </joint>
     <!-- =========================================== -->
-    <!-- ================ MONO CAMERA JOINTS ============ -->
+    <!-- ============== STEREO CAMERAS ============= -->
     <!-- =========================================== -->
-    <joint name="f_camera_joint" type="fixed">
-        <origin xyz="0.6525 0.0 0.6625" rpy="0 0 0"/>
+    <joint name="stereo_bar_joint" type="fixed">
+        <origin xyz="${bar_x} 0 ${bar_z}" rpy="0 0 0"/>
         <parent link="base_link"/>
-        <child link="f_camera_link"/>
+        <child link="stereo_bar_link"/>
     </joint>
-    <joint name="r_camera_joint" type="fixed">
-        <origin xyz="-0.6525 0.0 0.6625" rpy="0 0 ${pi}"/>
-        <parent link="base_link"/>
-        <child link="r_camera_link"/>
-    </joint>
-    <!-- Optical frames: sit at the lens (matches the 0.05 m sensor <pose> in
-         gazebo_sensors.xacro) with REP-103 axis rotation. -->
-    <joint name="f_camera_optical_joint" type="fixed">
-        <origin xyz="0.05 0 0" rpy="${-pi/2} 0 ${-pi/2}"/>
-        <parent link="f_camera_link"/>
-        <child link="f_camera_optical_link"/>
-    </joint>
-    <joint name="r_camera_optical_joint" type="fixed">
-        <origin xyz="0.05 0 0" rpy="${-pi/2} 0 ${-pi/2}"/>
-        <parent link="r_camera_link"/>
-        <child link="r_camera_optical_link"/>
-    </joint>
+    <xacro:macro name="camera_joints" params="side y">
+        <joint name="cam_${side}_joint" type="fixed">
+            <origin xyz="${cam_dx} ${y} 0" rpy="0 0 0"/>
+            <parent link="stereo_bar_link"/>
+            <child link="cam_${side}_link"/>
+        </joint>
+        <joint name="cam_${side}_optical_joint" type="fixed">
+            <origin xyz="0 0 0" rpy="${-pi/2} 0 ${-pi/2}"/>
+            <parent link="cam_${side}_link"/>
+            <child link="cam_${side}_optical_frame"/>
+        </joint>
+    </xacro:macro>
+    <xacro:camera_joints side="left"  y="${stereo_baseline/2}"/>
+    <xacro:camera_joints side="right" y="${-stereo_baseline/2}"/>
     <!-- =========================================== -->
-    <!-- ============== IMU + GPS JOINTS =========== -->
+    <!-- ================ IMU / GPS ================ -->
     <!-- =========================================== -->
-    <!-- IMU near the whole-robot CoM (base_link inertial origin). -->
     <joint name="imu_joint" type="fixed">
-        <origin xyz="0 0 0.486" rpy="0 0 0"/>
+        <origin xyz="${imu_x} 0 ${imu_z}" rpy="0 0 0"/>
         <parent link="base_link"/>
         <child link="imu_link"/>
     </joint>
-    <!-- GPS antenna on top of the chassis (top face is z = 0.636), slightly
-         aft so it clears the cameras' view. -->
     <joint name="gps_joint" type="fixed">
-        <origin xyz="-0.2 0 0.636" rpy="0 0 0"/>
+        <origin xyz="${gps_x} 0 ${gps_z}" rpy="0 0 0"/>
         <parent link="base_link"/>
         <child link="gps_link"/>
